File: KiCAD 7.0/Teensy-RV-Leveling-Helper-v1.kicad_sch (KiCad schematic)
At the start: 12 parts, among them J1 Conn_01x04_Pin, Q1 2N3904, Q2 2N3906, U1 Powerboost1000C, U2 Teensy4.0, U3 BMA400, U4 Teensy ILI9341

Commit message: Add files via upload
Parts:
- removed J1: Conn_01x04_Pin, symbol Connector:Conn_01x04_Pin
Connections:
- net USB VCC is gone; now on net USB VIN: U1.1 (USB)
- net DISABLE IN: now reaches U1.4 (EN)
- net BATT VDD: no longer names the net of U1.2 (BAT)
Changed lines of the file:
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@@
   (junction (at 68.58 106.68) (diameter 0) (color 0 0 0 0)
   )
-  (junction (at 27.94 41.91) (diameter 0) (color 0 0 0 0)
-  )
   (junction (at 173.99 128.27) (diameter 0) (color 0 0 0 0)
   )
@@
   )
   (junction (at 229.87 133.35) (diameter 0) (color 0 0 0 0)
-  )
-  (junction (at 30.48 36.83) (diameter 0) (color 0 0 0 0)
   )
   (no_connect (at 110.49 39.37))
@@
   (no_connect (at 166.37 67.31))
   (no_connect (at 166.37 64.77))
-  (no_connect (at 31.75 62.23))
   (no_connect (at 45.72 71.12))
   (no_connect (at 166.37 97.79))
@@
   (no_connect (at 149.86 45.72))
   (no_connect (at 166.37 41.91))
+  (no_connect (at 31.75 58.42))
   (no_connect (at 166.37 72.39))
   (no_connect (at 166.37 31.75))
@@
     (stroke (width 0) (type default))
   )
+  (wire (pts (xy 30.48 44.45) (xy 62.23 44.45))
+    (stroke (width 0) (type default))
+  )
   (wire (pts (xy 100.33 133.35) (xy 229.87 133.35))
     (stroke (width 0) (type default))
@@
     (stroke (width 0) (type default))
   )
-  (wire (pts (xy 54.61 19.05) (xy 54.61 34.29))
-    (stroke (width 0) (type default))
-  )
   (wire (pts (xy 44.45 119.38) (xy 68.58 119.38))
     (stroke (width 0) (type default))
   )
-  (wire (pts (xy 46.99 30.48) (xy 62.23 30.48))
+  (wire (pts (xy 46.99 31.75) (xy 57.15 31.75))
     (stroke (width 0) (type default))
   )
@@
     (stroke (width 0) (type default))
   )
+  (wire (pts (xy 25.4 39.37) (xy 57.15 39.37))
+    (stroke (width 0) (type default))
+  )
+  (wire (pts (xy 25.4 39.37) (xy 25.4 62.23))
+    (stroke (width 0) (type default))
+  )
   (wire (pts (xy 176.53 125.73) (xy 214.63 125.73))
     (stroke (width 0) (type default))
   )
-  (wire (pts (xy 30.48 36.83) (xy 30.48 54.61))
-    (stroke (width 0) (type default))
-  )
   (wire (pts (xy 166.37 95.25) (xy 173.99 95.25))
     (stroke (width 0) (type default))
@@
     (stroke (width 0) (type default))
   )
-  (wire (pts (xy 46.99 26.67) (xy 59.69 26.67))
-    (stroke (width 0) (type default))
-  )
-  (wire (pts (xy 27.94 58.42) (xy 31.75 58.42))
-    (stroke (width 0) (type default))
-  )
   (wire (pts (xy 95.25 62.23) (xy 110.49 62.23))
     (stroke (width 0) (type default))
@@
     (stroke (width 0) (type default))
   )
-  (wire (pts (xy 30.48 36.83) (xy 57.15 36.83))
-    (stroke (width 0) (type default))
-  )
   (wire (pts (xy 20.32 110.49) (xy 27.94 110.49))
     (stroke (width 0) (type default))
@@
     (stroke (width 0) (type default))
   )
-  (wire (pts (xy 27.94 41.91) (xy 62.23 41.91))
-    (stroke (width 0) (type default))
-  )
   (wire (pts (xy 100.33 80.01) (xy 110.49 80.01))
     (stroke (width 0) (type default))
@@
     (stroke (width 0) (type default))
   )
-  (wire (pts (xy 25.4 36.83) (xy 30.48 36.83))
-    (stroke (width 0) (type default))
-  )
   (wire (pts (xy 214.63 119.38) (xy 214.63 125.73))
     (stroke (width 0) (type default))
@@
     (stroke (width 0) (type default))
   )
-  (wire (pts (xy 46.99 19.05) (xy 54.61 19.05))
+  (wire (pts (xy 57.15 31.75) (xy 57.15 39.37))
+    (stroke (width 0) (type default))
+  )
+  (wire (pts (xy 46.99 26.67) (xy 62.23 26.67))
     (stroke (width 0) (type default))
   )
@@
     (stroke (width 0) (type default))
   )
-  (wire (pts (xy 25.4 41.91) (xy 27.94 41.91))
-    (stroke (width 0) (type default))
-  )
   (wire (pts (xy 95.25 138.43) (xy 227.33 138.43))
     (stroke (width 0) (type default))
@@
     (stroke (width 0) (type default))
   )
-  (wire (pts (xy 25.4 39.37) (xy 59.69 39.37))
-    (stroke (width 0) (type default))
-  )
   (wire (pts (xy 27.94 110.49) (xy 29.21 110.49))
     (stroke (width 0) (type default))
@@
     (stroke (width 0) (type default))
   )
-  (wire (pts (xy 46.99 22.86) (xy 57.15 22.86))
-    (stroke (width 0) (type default))
-  )
   (wire (pts (xy 68.58 106.68) (xy 68.58 107.95))
     (stroke (width 0) (type default))
@@
     (stroke (width 0) (type default))
   )
-  (wire (pts (xy 27.94 41.91) (xy 27.94 58.42))
-    (stroke (width 0) (type default))
-  )
   (wire (pts (xy 80.01 85.09) (xy 80.01 128.27))
     (stroke (width 0) (type default))
   )
-  (wire (pts (xy 25.4 34.29) (xy 54.61 34.29))
+  (wire (pts (xy 25.4 62.23) (xy 31.75 62.23))
     (stroke (width 0) (type default))
   )
@@
     (stroke (width 0) (type default))
   )
+  (wire (pts (xy 30.48 44.45) (xy 30.48 54.61))
+    (stroke (width 0) (type default))
+  )
   (wire (pts (xy 232.41 119.38) (xy 232.41 125.73))
     (stroke (width 0) (type default))
   )
+  (wire (pts (xy 62.23 26.67) (xy 62.23 44.45))
+    (stroke (width 0) (type default))
+  )
   (wire (pts (xy 68.58 119.38) (xy 68.58 115.57))
     (stroke (width 0) (type default))
@@
     (stroke (width 0) (type default))
   )
-  (wire (pts (xy 57.15 22.86) (xy 57.15 36.83))
-    (stroke (width 0) (type default))
-  )
   (wire (pts (xy 184.15 55.88) (xy 184.15 109.22))
     (stroke (width 0) (type default))
@@
     (stroke (width 0) (type default))
   )
-  (wire (pts (xy 62.23 30.48) (xy 62.23 41.91))
-    (stroke (width 0) (type default))
-  )
   (wire (pts (xy 222.25 119.38) (xy 222.25 128.27))
     (stroke (width 0) (type default))
@@
     (stroke (width 0) (type default))
   )
-  (wire (pts (xy 59.69 26.67) (xy 59.69 39.37))
-    (stroke (width 0) (type default))
-  )
   (wire (pts (xy 102.87 82.55) (xy 110.49 82.55))
     (stroke (width 0) (type default))
@@
     (stroke (width 0) (type default))
   )
-  (global_label "BATT IN" (shape input) (at 46.99 26.67 180) (fields_autoplaced)
+  (global_label "DISABLE IN" (shape input) (at 46.99 31.75 180) (fields_autoplaced)
     (effects (font (size 1.27 1.27)) (justify right))
-    (property "Intersheetrefs" "${INTERSHEET_REFS}" (at 36.8875 26.67 0)
+    (property "Intersheetrefs" "${INTERSHEET_REFS}" (at 33.5613 31.75 0)
       (effects (font (size 1.27 1.27)) (justify right) hide)
     )
   )
-  (global_label "USB VCC" (shape input) (at 46.99 22.86 180) (fields_autoplaced)
+  (global_label "USB VIN" (shape input) (at 46.99 26.67 180) (fields_autoplaced)
     (effects (font (size 1.27 1.27)) (justify right))
-    (property "Intersheetrefs" "${INTERSHEET_REFS}" (at 35.678 22.86 0)
-      (effects (font (size 1.27 1.27)) (justify right) hide)
-    )
-  )
-  (global_label "BATT VDD" (shape input) (at 46.99 30.48 180) (fields_autoplaced)
-    (effects (font (size 1.27 1.27)) (justify right))
-    (property "Intersheetrefs" "${INTERSHEET_REFS}" (at 35.1942 30.48 0)
-      (effects (font (size 1.27 1.27)) (justify right) hide)
-    )
-  )
-  (global_label "USB VIN" (shape input) (at 46.99 19.05 180) (fields_autoplaced)
-    (effects (font (size 1.27 1.27)) (justify right))
-    (property "Intersheetrefs" "${INTERSHEET_REFS}" (at 36.2827 19.05 0)
+    (property "Intersheetrefs" "${INTERSHEET_REFS}" (at 36.2827 27.94 0)
       (effects (font (size 1.27 1.27)) (justify right) hide)
     )
@@
         )
       )
-    )
-  )
-  (symbol (lib_id "Connector:Conn_01x04_Pin") (at 20.32 36.83 0) (unit 1)
-    (in_bom yes) (on_board yes) (dnp no)
-    (property "Reference" "J1" (at 21.59 27.94 0)
-      (effects (font (size 1.27 1.27)))
-    )
-    (property "Value" "Conn_01x04_Pin" (at 21.59 30.48 0)
-      (effects (font (size 1.27 1.27)))
-    )
-    (property "Footprint" "" (at 20.32 36.83 0)
-      (effects (font (size 1.27 1.27)) hide)
-    )
-    (property "Datasheet" "~" (at 20.32 36.83 0)
-      (effects (font (size 1.27 1.27)) hide)
-    )
-    (pin "1")
-    (pin "2")
-    (pin "3")
-    (pin "4")
-    (instances
-      (project "Teensy-RV-Leveling-Helper-v1"
-        (path "/40e83549-3702-4fa9-b9ab-1c775b6c5471"
-          (reference "J1") (unit 1)
-        )
-      )

Commit message: Add files via upload
Updated to include new PCB
Parts:
- added H1: USB-a, MountingHole:MountingHole_2.5mm, symbol Mechanical:MountingHole
- added H2: USB-b, MountingHole:MountingHole_2.5mm, symbol Mechanical:MountingHole
- added H3: USB-c, MountingHole:MountingHole_2.5mm, symbol Mechanical:MountingHole
- added H4: USB-d, MountingHole:MountingHole_2.5mm, symbol Mechanical:MountingHole
- added H5: PCB-a, MountingHole:MountingHole_2.7mm_M2.5_Pad_TopBottom, symbol Mechanical:MountingHole_Pad
- added H6: PCB-b, MountingHole:MountingHole_2.7mm_M2.5_Pad_TopBottom, symbol Mechanical:MountingHole_Pad
- added H7: PCB-c, MountingHole:MountingHole_2.7mm_M2.5_Pad_TopBottom, symbol Mechanical:MountingHole_Pad
- added H8: PCB-d, MountingHole:MountingHole_2.7mm_M2.5_Pad_TopBottom, symbol Mechanical:MountingHole_Pad
- added J1: USB VIN, Connector_PinHeader_2.54mm:PinHeader_1x01_P2.54mm_Vertical, symbol Connector_Generic:Conn_01x01
- added J2: DISABLE SW, Connector_PinHeader_2.54mm:PinHeader_1x02_P2.54mm_Vertical, symbol Connector_Generic:Conn_01x02
- U1: footprint (none) -> MJC:PowerBoost1000C
- U2: footprint (none) -> teensy:Teensy40
- U3: footprint (none) -> MJC:BMA400
- U4: footprint (none) -> MJC:ILI9341
Connections:
- net GNDREF: now also U1.7 (G), U3.1 (GND), U4.2 (GND), H5.1, H6.1, H7.1, H8.1, J2.2 (Pin_2); no longer U3. (SDA/PICO), U4. (VCC)
- net at R5.2, U1.8 (5Vo), U2.33 (VIN): now also U4.1 (VCC), U4.8 (LED); no longer U4. (VCC)
- net at Q2.1 (E), R8.2, U2.31 (3V3): now also U3.2 (3V3), U4.4 (RESET); no longer U3. (SDA/PICO), U4. (VCC)
- net at U2.11 (9_OUT1C): now also U4.5 (DC); no longer U4. (VCC)
- net at U2.13 (11_MOSI_CTX1): now also U4.12 (T_DIN), U4.6 (SDI(MOSI)); no longer U4. (VCC)
- net at U2.14 (12_MISO_MQSL): now also U4.13 (T_DO), U4.9 (SDO(MISO)); no longer U4. (VCC)
- net at U2.20 (13_SCK_CRX1_LED): now also U4.10 (T_CLK), U4.7 (SCK); no longer U4. (VCC)
- net at U2.21 (14_A0_TX3_SPDIF_OUT): now also U4.3 (CS); no longer U4. (VCC)
- net at U2.7 (5_IN2): now also U4.11 (T_CS); no longer U4. (VCC)
- net at U2.25 (18_A4_SDA0): now also U3.3 (SDA/PICO); no longer U3. (SDA/PICO)
- net at U2.26 (19_A5_SCL0): now also U3.4 (SCL/SCK); no longer U3. (SDA/PICO)
- net DISABLE IN: no longer names the net of U1.4 (EN)
- net DISABLE IN: now also J2.1 (Pin_1)
- net USB VIN: no longer names the net of U1.1 (USB)
- net USB VIN: now also J1.1 (Pin_1)
- no-connect marks 54 -> 53
